Commit message: big update

File: model/urdf/sawyer_gripper_mujoco.urdf (robot description, URDF)
Before this commit: robot sawyer, 27 links, 26 joints
Links:
- removed link gripah_base
- removed link narrow_finger_link
- removed link wide_finger_link
- added link right_connector_plate_base, mass 0.0; collision cylinder length=0.0302 radius=0.04; visual mesh filename=package://intera_tools_description/meshes/connector_plate/c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
- added link right_connector_plate_mount
- added link right_electric_gripper_base, mass 2e-06; collision cylinder length=0.1 radius=0.029; visual mesh filename=package://intera_tools_description/meshes/electric_gripper/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
- added link right_gripper_base, mass 0.47
- added link right_gripper_l_finger, mass 0.001; collision box size=0.01 0.0135 0.075; collision box size=0.01 0.05 0.017
- added link right_gripper_l_finger_tip, mass 0.001; collision box size=0.016 0.007 0.037; visual mesh filename=package://intera_tools_description/meshes/electric_gripper/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
- added link right_gripper_r_finger, mass 0.001; collision box size=0.01 0.0135 0.075; collision box size=0.01 0.05 0.017
- added link right_gripper_r_finger_tip, mass 0.001; collision box size=0.016 0.007 0.037; visual mesh filename=package://intera_tools_description/meshes/electric_gripper/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
- added link right_gripper_tip, mass 2e-06
- link head: geometry collision sphere radius=0.18; visual mesh filename=package://sawyer_description/meshes/sawyer_pv/head.STL
Joints:
- removed joint narrow_finger_joint
- removed joint wide_finger_joint
- added joint right_connector_plate_base_joint: type fixed, parent right_gripper_base, child right_connector_plate_base, origin xyz=0 0 0.0018 rpy=0 0 0
- added joint right_connector_plate_mount_joint: type fixed, parent right_connector_plate_base, child right_connector_plate_mount, origin xyz=0 0 0.0176 rpy=0 0 0
- added joint right_electric_gripper_base_joint: type fixed, parent right_connector_plate_mount, child right_electric_gripper_base, origin xyz=0 0 0 rpy=0 0 0
- added joint right_gripper_l_finger_joint: type prismatic, parent right_electric_gripper_base, child right_gripper_l_finger, origin xyz=0.003 -0.0015 0.04552 rpy=0 0 0, axis 0 1 0, limit lower=0.0 upper=0.020833 effort=20.0 velocity=5.0
- added joint right_gripper_l_finger_tip_joint: type fixed, parent right_gripper_l_finger, child right_gripper_l_finger_tip, origin xyz=0.0 0.01725 0.075 rpy=0 0 0
- added joint right_gripper_r_finger_joint: type prismatic, parent right_electric_gripper_base, child right_gripper_r_finger, origin xyz=0.003 0.0015 0.04552 rpy=0 0 0, axis 0 1 0, limit lower=-0.020833 upper=0.0 effort=20.0 velocity=5.0, mimic joint=right_gripper_l_finger_joint multiplier=-1.0
- added joint right_gripper_r_finger_tip_joint: type fixed, parent right_gripper_r_finger, child right_gripper_r_finger_tip, origin xyz=0.0 -0.01725 0.075 rpy=0 0 0
- added joint right_gripper_tip_joint: type fixed, parent right_gripper_base, child right_gripper_tip, origin xyz=0 0 0.14062 rpy=0 0 0
- joint right_gripper_base_joint: child gripah_base -> right_gripper_base; origin xyz=0 0 0.025 rpy=-1.5707 0 0 -> xyz=0 0 -0.005 rpy=0 0 0

File: model/urdf/sawyer_mujoco.urdf.xacro (robot description, xacro)
@@ -1,4 +1,7 @@
 <?xml version="1.0" ?>
 <robot name="sawyer" xmlns:xacro="http://www.ros.org/wiki/xacro">
+  <mujoco>
+     <compiler meshdir="/home/tarik/sawyer_mujoco/meshes/" balanceinertia="true" discardvisual="false"/>
+  </mujoco>
   <xacro:arg name="gazebo" default="false"/>
   <xacro:arg name="pedestal" default="true"/>
